Commit message: 关节阻尼和摩擦改为原来的5倍

File: robots/descriptions/go2_description/xacro/const.xacro (robot description, xacro)
@@ -39,6 +39,6 @@
     <xacro:property name="calf_offset_z" value="-0.213"/>
     <!-- joint limits -->
-    <xacro:property name="damping" value="0.01"/>
-    <xacro:property name="friction" value="0.2"/>
+    <xacro:property name="damping" value="0.05"/>
+    <xacro:property name="friction" value="1.0"/>
     <xacro:property name="hip_position_max" value="1.0472"/>
     <xacro:property name="hip_position_min" value="-1.0472"/>
